File: hardware/v2/powerboard/powerboard.kicad_pcb (KiCad board)
At the start: 2 copper layers, 52.7 x 66 mm, 35 parts, among them J1 LEG1_PWR, J10 UBEC3, J11 SBEC, J12 LOGIC_5V_OUT, J13 MONITOR, J2 LEG2_PWR, J3 LEG3_PWR, J4 LEG4_PWR, J5 LEG5_PWR, J6 LEG6_PWR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

Commit message: powerboard layout
Parts:
- added ON / OFF: MASTER_SW, Custom:SW_Slide_SPDT_Straight, F.Cu at (82.4, 128.6)
- moved J6 91.1 mm to (142.2, 71.1), turned to 90 degrees
- moved J5 83.7 mm to (134.6, 57.1), turned to 180 degrees
- moved J13 83.7 mm to (97.8, 128.3), turned to 90 degrees
- moved Q1 75.9 mm to (87.6, 99.1), turned to 180 degrees
- moved Q2 75.8 mm to (111.8, 99.1), turned to 180 degrees
- moved R4 72.6 mm to (125.7, 83.5), turned to 90 degrees
- moved R3 68.6 mm to (115.6, 83.5), turned to 90 degrees
- moved C3 68.4 mm to (131.9, 69.8), turned to 180 degrees
- moved J12 66.0 mm to (129.5, 82.5), turned to 180 degrees
- moved R2 64.6 mm to (101.6, 83.5), turned to 90 degrees
- moved R1 63.8 mm to (88.9, 83.6), turned to 90 degrees
- moved J11 62.1 mm to (121.9, 92.6), turned to 90 degrees
- moved R5 60.1 mm to (77.1, 92.7)
- moved J4 56.7 mm to (107.9, 57.1), turned to 180 degrees
- moved R7 56.5 mm to (72.4, 94.9), turned to 90 degrees
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Routing:
- net GND: track 223.6 -> 0.00 mm
- net VSERVO3: track 108.0 -> 0.00 mm
- net VSERVO2: track 105.5 -> 0.00 mm, vias 2 -> 0
- net VSERVO1: track 98.0 -> 0.00 mm, vias 2 -> 0
- net +VMAIN: track 86.8 -> 0.00 mm
- net +5V: track 62.7 -> 0.00 mm, vias 1 -> 0
- net PMOS_GATE_DRV: track 53.0 -> 0.00 mm, vias 2 -> 0
- net BATT_FUSED: track 47.7 -> 0.00 mm, vias 1 -> 0
- net PMOS_GATE: track 43.2 -> 2.54 mm
- net LED_U2: track 35.4 -> 0.00 mm
- net LED_U3: track 33.9 -> 0.00 mm, vias 2 -> 0
- net NPN_BASE: track 29.9 -> 0.00 mm, vias 2 -> 0
- net LED_SBEC: track 26.3 -> 0.00 mm
- net BATT_RAW: track 25.6 -> 0.00 mm
- net LED_U1: track 25.3 -> 0.00 mm
Other:
- board size 52.7 x 66 mm -> 101.6 x 81.9 mm

Commit message: powerboard layout adjustments
Parts:
- moved J13 28.7 mm to (91.4, 100.3)
- moved Q1 3.81 mm to (83.8, 99.1)
- moved Q2 1.27 mm to (113.0, 99.1)
Changed lines of the file:
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@@
 	(footprint "Capacitor_THT:CP_Radial_D13.0mm_P5.00mm"
 		(layer "F.Cu")
-		(at 131.855216 69.85 180)
+		(at 131.8552 69.85 180)
 		(descr "CP, Radial series, Radial, pin pitch=5.00mm, diameter=13mm, height=20mm, Electrolytic Capacitor")
 		(tags "CP Radial series Radial pin pitch 5.00mm diameter 13mm height 20mm Electrolytic Capacitor")
@@
 	(footprint "Package_TO_SOT_THT:TO-220-3_Vertical"
 		(layer "F.Cu")
-		(at 111.76 99.06 180)
+		(at 113.03 99.06 180)
 		(descr "TO-220-3, Vertical, RM 2.54mm, see https://www.vishay.com/docs/66542/to-220-1.pdf, generated with kicad-footprint-generator TO_SOT_THT_generate.py")
 		(tags "TO-220-3 Vertical RM 2.54mm")
@@
 	(footprint "Connector_PinHeader_2.54mm:PinHeader_1x05_P2.54mm_Vertical"
 		(layer "F.Cu")
-		(at 97.79 128.27 90)
+		(at 91.44 100.33 90)
 		(descr "Through hole straight pin header, 1x05, 2.54mm pitch, single row")
 		(tags "Through hole pin header THT 1x05 2.54mm single row")
@@
 	(footprint "Package_TO_SOT_THT:TO-220-3_Vertical"
 		(layer "F.Cu")
-		(at 87.63 99.06 180)
+		(at 83.82 99.06 180)
 		(descr "TO-220-3, Vertical, RM 2.54mm, see https://www.vishay.com/docs/66542/to-220-1.pdf, generated with kicad-footprint-generator TO_SOT_THT_generate.py")
 		(tags "TO-220-3 Vertical RM 2.54mm")
@@
 	(footprint "Capacitor_THT:CP_Radial_D13.0mm_P5.00mm"
 		(layer "F.Cu")
-		(at 101.375216 69.85 180)
+		(at 101.3752 69.85 180)
 		(descr "CP, Radial series, Radial, pin pitch=5.00mm, diameter=13mm, height=20mm, Electrolytic Capacitor")
 		(tags "CP Radial series Radial pin pitch 5.00mm diameter 13mm height 20mm Electrolytic Capacitor")

Commit message: powerboard rc1
Parts:
- moved R7 5.24 mm to (73.7, 100.0)
- moved R8 4.81 mm to (66.4, 90.2)
- moved C5 3.00 mm to (72.4, 83.8)
- moved D2 2.58 mm to (91.4, 79.7)
- moved R1 2.58 mm to (91.5, 83.5)
- moved Q3 1.64 mm to (71.5, 90.2), turned to 0 degrees
Routing:
- net BATT_FUSED: track 0.00 -> 142.9 mm
- net VSERVO1: track 0.00 -> 104.4 mm
- net VSERVO3: track 0.00 -> 77.9 mm
- net +VMAIN: track 0.00 -> 70.3 mm
- net VSERVO2: track 0.00 -> 64.3 mm
- net PMOS_GATE: track 2.54 -> 62.9 mm
- net SW_CTRL: track 0.00 -> 34.4 mm
- net BATT_RAW: track 0.00 -> 17.0 mm
- net NPN_BASE: track 0.00 -> 15.3 mm
- net PMOS_GATE_DRV: track 0.00 -> 13.4 mm
- net +5V: track 0.00 -> 8.44 mm
- net LED_U2: track 0.00 -> 1.96 mm
- net LED_U3: track 0.00 -> 1.94 mm
- net LED_SBEC: track 0.00 -> 1.94 mm
- added copper zone on B.Cu, net GND
- added copper zone on F.Cu, net GND
