File: hardware/v2/powerboard/powerboard.kicad_pcb (KiCad board)
At the start: 2 copper layers, 101.6 x 81.9 mm, 36 parts, among them J1 LEG1_PWR, J10 UBEC3, J11 SBEC, J12 LOGIC_5V_OUT, J13 MONITOR, J2 LEG2_PWR, J3 LEG3_PWR, J4 LEG4_PWR, J5 LEG5_PWR, J6 LEG6_PWR, J7 BATTERY, J8 UBEC1, J9 UBEC2, Q1 FQP47P06, Q2 FQP47P06, Q3 MMBT3904

Commit message: powerboard updates
Parts:
- F1: value 20A -> 3413.0331.22 20A; footprint Custom:Fuse Holder Mini -> Fuse:Fuse_1206_3216Metric; moved to B.Cu
- J10, J11, J8, J9: footprint Connector_Wire:SolderWire-0.25sqmm_1x04_P4.2mm_D0.65mm_OD1.7mm -> Custom:SolderWirePad_4x01_SMD_3x4mm
- Q1, Q2: value FQP47P06 -> IRF9540NPBF
- R5: value 100 -> 470
- SW1: renamed from ON / OFF
- moved F1 7.74 mm to (75.3, 69.3), turned to -90 degrees
- moved J11 6.59 mm to (120.9, 86.1)
- moved J8 6.48 mm to (85.3, 86.2)
- moved J10 6.46 mm to (110.7, 86.2)
- moved J9 6.40 mm to (97.6, 86.2)
- moved R5 2.57 mm to (79.0, 90.9)
- moved R1 1.29 mm to (90.6, 84.4)
- moved D2 1.17 mm to (90.6, 80.4)
- moved R2 1.15 mm to (102.7, 83.6)
- moved D3 1.09 mm to (102.7, 79.7)
Routing:
- net VSERVO1: track 104.4 -> 76.0 mm, vias 0 -> 1
- net VSERVO3: track 77.9 -> 97.7 mm, vias 0 -> 1
- net BATT_FUSED: track 142.9 -> 128.3 mm, vias 0 -> 1
- net BATT_RAW: track 17.0 -> 9.05 mm
- net +VMAIN: track 70.3 -> 64.3 mm
- net VSERVO2: track 64.3 -> 69.5 mm, vias 0 -> 1
- net LED_U1: track 0.00 -> 2.06 mm
- net PMOS_GATE_DRV: track 13.4 -> 14.6 mm
- net PMOS_GATE: track 62.9 -> 63.0 mm, vias 1 -> 2
- net GND: vias 0 -> 2
Other:
- board text added: "Hexabot Powerboard v2.1"
