File: hardware/v2/legboard/legboard.kicad_pcb (KiCad board)
At the start: 2 copper layers, 40.6 x 59.7 mm, 17 parts, among them J1 UPLINK_RJ11, J2 COXA, J3 FEMUR, J4 TIBIA, J5 SERVO_PWR_IN, U1 XIAO-RP2040, U2 SP3485CN, U3 INA4181A3IPWR

Commit message: hardware: fix legboard current-sense channel mapping, swap powerboard PMOS to IRF9540NPBF
Legboard: correct the INA4181 stub labels so U3 pins 2-4/13-15 map to
TOTAL/TIBIA current sensing per the corrected net table, instead of the
swapped TOTAL<->TIBIA assignment.

Powerboard: replace Q1/Q2 reverse-polarity PMOS (FQP47P06 -> IRF9540NPBF).
Parts:
- J2 Coxa: renamed from J2
- J3 Femur: renamed from J3
- J4 Tibia: renamed from J4
- turned R4 to 90 degrees
Connections:
- R2 pad 1: +6V_IN -> +6V
- R2 pad 2: ITOT_SP -> TIBIA_SP
- R2 pad 3: ITOT_SN -> TIBIA_SN
- R2 pad 4: +6V -> +6V_TIBIA
- R3 pad 2: COXA_SP -> FEMUR_SP
- R3 pad 3: COXA_SN -> FEMUR_SN
- R3 pad 4: +6V_COXA -> +6V_FEMUR
- R4 pad 1: +6V -> +6V_IN
- R4 pad 2: FEMUR_SP -> ITOT_SP
- R4 pad 3: FEMUR_SN -> ITOT_SN
- R4 pad 4: +6V_FEMUR -> +6V
- R5 pad 2: TIBIA_SP -> COXA_SP
- R5 pad 3: TIBIA_SN -> COXA_SN
- R5 pad 4: +6V_TIBIA -> +6V_COXA
- U1 pad 2: I_COXA_SENSE -> I_FEMUR_SENSE
- U1 pad 3: I_FEMUR_SENSE -> I_TIBIA_SENSE
- U1 pad 4: I_TIBIA_SENSE -> I_COXA_SENSE
- U3 pad 13: I_FEMUR_SENSE -> I_TOTAL_SENSE
- U3 pad 14: FEMUR_SN -> ITOT_SN
- U3 pad 15: FEMUR_SP -> ITOT_SP
- U3 pad 17: TIBIA_SP -> COXA_SP
- U3 pad 18: TIBIA_SN -> COXA_SN
- U3 pad 19: I_TIBIA_SENSE -> I_COXA_SENSE
- U3 pad 2: I_TOTAL_SENSE -> I_TIBIA_SENSE
- U3 pad 3: ITOT_SN -> TIBIA_SN
- U3 pad 4: ITOT_SP -> TIBIA_SP
- U3 pad 6: COXA_SP -> FEMUR_SP
- U3 pad 7: COXA_SN -> FEMUR_SN
- U3 pad 8: I_COXA_SENSE -> I_FEMUR_SENSE
Routing:
- net +6V: track 0.19 -> 81.2 mm, vias 0 -> 4
- net +3.3V: track 3.80 -> 64.5 mm, vias 0 -> 2
- net COXA_PWM: track 0.00 -> 53.7 mm, vias 0 -> 1
- net +5V: track 0.00 -> 49.4 mm
- net FEMUR_PWM: track 0.00 -> 35.8 mm
- net +6V_TIBIA: track 0.00 -> 34.8 mm
- net I_FEMUR_SENSE: track 0.00 -> 33.9 mm, vias 0 -> 2
- net RS485_A: track 0.00 -> 32.1 mm
- net +6V_IN: track 0.21 -> 32.1 mm, vias 0 -> 3
- net RS485_DE: track 0.00 -> 28.3 mm
- net RS485_B: track 0.00 -> 26.3 mm
- net TIBIA_PWM: track 0.00 -> 26.2 mm
- net +6V_COXA: track 0.00 -> 24.2 mm
- net GND: track 38.5 -> 60.7 mm, vias 4 -> 6
- net RP_TXD: track 0.00 -> 21.9 mm
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- added copper zone on B.Cu, net +6V_IN
- added copper zone on F.Cu, net +6V_IN
Other:
- board text added: "Legbord v2"
